File: schematic/devel/detector.sch (KiCad schematic (older format))
At the start: 20 parts

Commit message: made small adjustments, created netlist
Parts:
- gave numbers to parts that had none: 12
Changed lines of the file:
@@
 P 2550 3200
 AR Path="/5D92E8C4" Ref="D?"  Part="1"
-AR Path="/5D929D0E/5D92E8C4" Ref="D?"  Part="1"
-F 0 "D?" H 2450 3500 50  0000 L CNN
+AR Path="/5D929D0E/5D92E8C4" Ref="D5"  Part="1"
+F 0 "D5" H 2450 3500 50  0000 L CNN
 F 1 "S599x" H 2400 3400 50  0000 L CNN
 F 2 "" V 2650 3100 50  0001 C CNN
@@
 P 4850 2850
 AR Path="/5D92E8D7" Ref="R?"  Part="1"
-AR Path="/5D929D0E/5D92E8D7" Ref="R?"  Part="1"
-F 0 "R?" V 4654 2850 50  0000 C CNN
+AR Path="/5D929D0E/5D92E8D7" Ref="R4"  Part="1"
+F 0 "R4" V 4654 2850 50  0000 C CNN
 F 1 "100k" V 4745 2850 50  0000 C CNN
 F 2 "" H 4850 2850 50  0001 C CNN
@@
 P 4850 2450
 AR Path="/5D92E8DD" Ref="C?"  Part="1"
-AR Path="/5D929D0E/5D92E8DD" Ref="C?"  Part="1"
-F 0 "C?" V 4621 2450 50  0000 C CNN
+AR Path="/5D929D0E/5D92E8DD" Ref="C16"  Part="1"
+F 0 "C16" V 4621 2450 50  0000 C CNN
 F 1 "4p" V 4712 2450 50  0000 C CNN
 F 2 "" H 4850 2450 50  0001 C CNN
@@
 P 4850 3300
 AR Path="/5D92E8F0" Ref="U?"  Part="2"
-AR Path="/5D929D0E/5D92E8F0" Ref="U?"  Part="2"
-F 0 "U?" H 5000 3500 50  0000 C CNN
+AR Path="/5D929D0E/5D92E8F0" Ref="U4"  Part="2"
+F 0 "U4" H 5000 3500 50  0000 C CNN
 F 1 "OPA4197" H 4900 3600 50  0000 C CNN
 F 2 "" H 4850 3300 50  0001 C CNN
@@
 P 4850 4450
 AR Path="/5D92E904" Ref="R?"  Part="1"
-AR Path="/5D929D0E/5D92E904" Ref="R?"  Part="1"
-F 0 "R?" V 4654 4450 50  0000 C CNN
+AR Path="/5D929D0E/5D92E904" Ref="R5"  Part="1"
+F 0 "R5" V 4654 4450 50  0000 C CNN
 F 1 "100k" V 4745 4450 50  0000 C CNN
 F 2 "" H 4850 4450 50  0001 C CNN
@@
 P 4850 4050
 AR Path="/5D92E90A" Ref="C?"  Part="1"
-AR Path="/5D929D0E/5D92E90A" Ref="C?"  Part="1"
-F 0 "C?" V 4621 4050 50  0000 C CNN
+AR Path="/5D929D0E/5D92E90A" Ref="C17"  Part="1"
+F 0 "C17" V 4621 4050 50  0000 C CNN
 F 1 "4p" V 4712 4050 50  0000 C CNN
 F 2 "" H 4850 4050 50  0001 C CNN
@@
 P 4850 4900
 AR Path="/5D92E91D" Ref="U?"  Part="3"
-AR Path="/5D929D0E/5D92E91D" Ref="U?"  Part="3"
-F 0 "U?" H 5000 5100 50  0000 C CNN
+AR Path="/5D929D0E/5D92E91D" Ref="U4"  Part="3"
+F 0 "U4" H 5000 5100 50  0000 C CNN
 F 1 "OPA4197" H 4900 5200 50  0000 C CNN
 F 2 "" H 4850 4900 50  0001 C CNN
@@
 P 3150 2450
 AR Path="/5D92E932" Ref="C?"  Part="1"
-AR Path="/5D929D0E/5D92E932" Ref="C?"  Part="1"
-F 0 "C?" V 2921 2450 50  0000 C CNN
+AR Path="/5D929D0E/5D92E932" Ref="C14"  Part="1"
+F 0 "C14" V 2921 2450 50  0000 C CNN
 F 1 "4p" V 3012 2450 50  0000 C CNN
 F 2 "" H 3150 2450 50  0001 C CNN
@@
 P 3150 2850
 AR Path="/5D92E938" Ref="R?"  Part="1"
-AR Path="/5D929D0E/5D92E938" Ref="R?"  Part="1"
-F 0 "R?" V 2954 2850 50  0000 C CNN
+AR Path="/5D929D0E/5D92E938" Ref="R2"  Part="1"
+F 0 "R2" V 2954 2850 50  0000 C CNN
 F 1 "100k" V 3045 2850 50  0000 C CNN
 F 2 "" H 3150 2850 50  0001 C CNN
@@
 P 3150 3300
 AR Path="/5D92E94A" Ref="U?"  Part="1"
-AR Path="/5D929D0E/5D92E94A" Ref="U?"  Part="1"
-F 0 "U?" H 3300 3500 50  0000 C CNN
+AR Path="/5D929D0E/5D92E94A" Ref="U4"  Part="1"
+F 0 "U4" H 3300 3500 50  0000 C CNN
 F 1 "OPA4197" H 3200 3600 50  0000 C CNN
 F 2 "" H 3150 3300 50  0001 C CNN
@@
 P 3150 4900
 AR Path="/5D92E950" Ref="U?"  Part="4"
-AR Path="/5D929D0E/5D92E950" Ref="U?"  Part="4"
-F 0 "U?" H 3300 5100 50  0000 C CNN
+AR Path="/5D929D0E/5D92E950" Ref="U4"  Part="4"
+F 0 "U4" H 3300 5100 50  0000 C CNN
 F 1 "OPA4197" H 3200 5200 50  0000 C CNN
 F 2 "" H 3150 4900 50  0001 C CNN
@@
 P 3150 4050
 AR Path="/5D92E961" Ref="C?"  Part="1"
-AR Path="/5D929D0E/5D92E961" Ref="C?"  Part="1"
-F 0 "C?" V 2921 4050 50  0000 C CNN
+AR Path="/5D929D0E/5D92E961" Ref="C15"  Part="1"
+F 0 "C15" V 2921 4050 50  0000 C CNN
 F 1 "4p" V 3012 4050 50  0000 C CNN
 F 2 "" H 3150 4050 50  0001 C CNN
@@
 P 3150 4450
 AR Path="/5D92E967" Ref="R?"  Part="1"
-AR Path="/5D929D0E/5D92E967" Ref="R?"  Part="1"
-F 0 "R?" V 2954 4450 50  0000 C CNN
+AR Path="/5D929D0E/5D92E967" Ref="R3"  Part="1"
+F 0 "R3" V 2954 4450 50  0000 C CNN
 F 1 "100k" V 3045 4450 50  0000 C CNN
 F 2 "" H 3150 4450 50  0001 C CNN
@@
 P 1650 3750
 AR Path="/5D92E981" Ref="U?"  Part="5"
-AR Path="/5D929D0E/5D92E981" Ref="U?"  Part="5"
-F 0 "U?" V 1325 3750 50  0000 C CNN
+AR Path="/5D929D0E/5D92E981" Ref="U4"  Part="5"
+F 0 "U4" V 1325 3750 50  0000 C CNN
 F 1 "OPA4197" V 1416 3750 50  0000 C CNN
 F 2 "" H 1650 3750 50  0001 C CNN
@@
 P 1950 2700
 AR Path="/5D92E998" Ref="C?"  Part="1"
-AR Path="/5D929D0E/5D92E998" Ref="C?"  Part="1"
-F 0 "C?" V 1721 2700 50  0000 C CNN
+AR Path="/5D929D0E/5D92E998" Ref="C12"  Part="1"
+F 0 "C12" V 1721 2700 50  0000 C CNN
 F 1 "100n" V 1812 2700 50  0000 C CNN
 F 2 "" H 1950 2700 50  0001 C CNN
@@
 P 1950 4850
 AR Path="/5D92E9AA" Ref="C?"  Part="1"
-AR Path="/5D929D0E/5D92E9AA" Ref="C?"  Part="1"
-F 0 "C?" V 1721 4850 50  0000 C CNN
+AR Path="/5D929D0E/5D92E9AA" Ref="C13"  Part="1"
+F 0 "C13" V 1721 4850 50  0000 C CNN
 F 1 "100n" V 1812 4850 50  0000 C CNN
 F 2 "" H 1950 4850 50  0001 C CNN
@@
 $EndComp
 $Comp
-L Sensor_OpticalPosition:S599x D?
+L Sensor_OpticalPosition:S599x D5
 U 2 1 5D9B96B5
 P 4250 3200
-F 0 "D?" H 4257 3495 50  0000 C CNN
+F 0 "D5" H 4257 3495 50  0000 C CNN
 F 1 "S599x" H 4257 3404 50  0000 C CNN
 F 2 "" H 4200 3200 50  0001 C CNN
@@
 Connection ~ 4450 3200
 $Comp
-L Sensor_OpticalPosition:S599x D?
+L Sensor_OpticalPosition:S599x D5
 U 3 1 5D9D0743
 P 4250 4800
-F 0 "D?" H 4257 5095 50  0000 C CNN
+F 0 "D5" H 4257 5095 50  0000 C CNN
 F 1 "S599x" H 4257 5004 50  0000 C CNN
 F 2 "" H 4200 4800 50  0001 C CNN
@@
 Connection ~ 4450 4800
 $Comp
-L Sensor_OpticalPosition:S599x D?
+L Sensor_OpticalPosition:S599x D5
 U 4 1 5D9ED07A
 P 2550 4800
-F 0 "D?" H 2557 5095 50  0000 C CNN
+F 0 "D5" H 2557 5095 50  0000 C CNN
 F 1 "S599x" H 2557 5004 50  0000 C CNN
 F 2 "" H 2500 4800 50  0001 C CNN
@@
 TRANSIMPEDANCE AMPLIFIER
 $Comp
-L Sensor_OpticalPosition:S599x D?
+L Sensor_OpticalPosition:S599x D5
 U 5 1 5D9F663F
 P 8500 3850
-F 0 "D?" H 8558 3936 50  0000 L CNN
+F 0 "D5" H 8558 3936 50  0000 L CNN
 F 1 "S599x" H 8558 3845 50  0000 L CNN
 F 2 "" H 8450 3850 50  0001 C CNN

Commit message: assigned footprints to symbols
Parts:
- C12, C13: footprint (none) -> Capacitor_SMD:C_0603_1608Metric
- C14, C15, C16, C17: footprint (none) -> Capacitor_SMD:C_0402_1005Metric
- R2, R3, R4, R5: footprint (none) -> Resistor_SMD:R_0805_2012Metric
- U4: footprint (none) -> Package_SO:MSOP-8_3x3mm_P0.65mm
Changed lines of the file:
@@
 F 0 "R4" V 4654 2850 50  0000 C CNN
 F 1 "100k" V 4745 2850 50  0000 C CNN
-F 2 "" H 4850 2850 50  0001 C CNN
+F 2 "Resistor_SMD:R_0805_2012Metric" H 4850 2850 50  0001 C CNN
 F 3 "~" H 4850 2850 50  0001 C CNN
 	1    4850 2850
@@
 F 0 "C16" V 4621 2450 50  0000 C CNN
 F 1 "4p" V 4712 2450 50  0000 C CNN
-F 2 "" H 4850 2450 50  0001 C CNN
+F 2 "Capacitor_SMD:C_0402_1005Metric" H 4850 2450 50  0001 C CNN
 F 3 "~" H 4850 2450 50  0001 C CNN
 	1    4850 2450
@@
 F 0 "U4" H 5000 3500 50  0000 C CNN
 F 1 "OPA4197" H 4900 3600 50  0000 C CNN
-F 2 "" H 4850 3300 50  0001 C CNN
+F 2 "Package_SO:MSOP-8_3x3mm_P0.65mm" H 4850 3300 50  0001 C CNN
 F 3 "~" H 4850 3300 50  0001 C CNN
 	2    4850 3300
@@
 F 0 "R5" V 4654 4450 50  0000 C CNN
 F 1 "100k" V 4745 4450 50  0000 C CNN
-F 2 "" H 4850 4450 50  0001 C CNN
+F 2 "Resistor_SMD:R_0805_2012Metric" H 4850 4450 50  0001 C CNN
 F 3 "~" H 4850 4450 50  0001 C CNN
 	1    4850 4450
@@
 F 0 "C17" V 4621 4050 50  0000 C CNN
 F 1 "4p" V 4712 4050 50  0000 C CNN
-F 2 "" H 4850 4050 50  0001 C CNN
+F 2 "Capacitor_SMD:C_0402_1005Metric" H 4850 4050 50  0001 C CNN
 F 3 "~" H 4850 4050 50  0001 C CNN
 	1    4850 4050
@@
 F 0 "U4" H 5000 5100 50  0000 C CNN
 F 1 "OPA4197" H 4900 5200 50  0000 C CNN
-F 2 "" H 4850 4900 50  0001 C CNN
+F 2 "Package_SO:MSOP-8_3x3mm_P0.65mm" H 4850 4900 50  0001 C CNN
 F 3 "~" H 4850 4900 50  0001 C CNN
 	3    4850 4900
@@
 F 0 "C14" V 2921 2450 50  0000 C CNN
 F 1 "4p" V 3012 2450 50  0000 C CNN
-F 2 "" H 3150 2450 50  0001 C CNN
+F 2 "Capacitor_SMD:C_0402_1005Metric" H 3150 2450 50  0001 C CNN
 F 3 "~" H 3150 2450 50  0001 C CNN
 	1    3150 2450
@@
 F 0 "R2" V 2954 2850 50  0000 C CNN
 F 1 "100k" V 3045 2850 50  0000 C CNN
-F 2 "" H 3150 2850 50  0001 C CNN
+F 2 "Resistor_SMD:R_0805_2012Metric" H 3150 2850 50  0001 C CNN
 F 3 "~" H 3150 2850 50  0001 C CNN
 	1    3150 2850
@@
 F 0 "U4" H 3300 3500 50  0000 C CNN
 F 1 "OPA4197" H 3200 3600 50  0000 C CNN
-F 2 "" H 3150 3300 50  0001 C CNN
+F 2 "Package_SO:MSOP-8_3x3mm_P0.65mm" H 3150 3300 50  0001 C CNN
 F 3 "~" H 3150 3300 50  0001 C CNN
 	1    3150 3300
@@
 F 0 "U4" H 3300 5100 50  0000 C CNN
 F 1 "OPA4197" H 3200 5200 50  0000 C CNN
-F 2 "" H 3150 4900 50  0001 C CNN
+F 2 "Package_SO:MSOP-8_3x3mm_P0.65mm" H 3150 4900 50  0001 C CNN
 F 3 "~" H 3150 4900 50  0001 C CNN
 	4    3150 4900
@@
 F 0 "C15" V 2921 4050 50  0000 C CNN
 F 1 "4p" V 3012 4050 50  0000 C CNN
-F 2 "" H 3150 4050 50  0001 C CNN
+F 2 "Capacitor_SMD:C_0402_1005Metric" H 3150 4050 50  0001 C CNN
 F 3 "~" H 3150 4050 50  0001 C CNN
 	1    3150 4050
@@
 F 0 "R3" V 2954 4450 50  0000 C CNN
 F 1 "100k" V 3045 4450 50  0000 C CNN
-F 2 "" H 3150 4450 50  0001 C CNN
+F 2 "Resistor_SMD:R_0805_2012Metric" H 3150 4450 50  0001 C CNN
 F 3 "~" H 3150 4450 50  0001 C CNN
 	1    3150 4450
@@
 F 0 "U4" V 1325 3750 50  0000 C CNN
 F 1 "OPA4197" V 1416 3750 50  0000 C CNN
-F 2 "" H 1650 3750 50  0001 C CNN
+F 2 "Package_SO:MSOP-8_3x3mm_P0.65mm" H 1650 3750 50  0001 C CNN
 F 3 "~" H 1650 3750 50  0001 C CNN
 	5    1650 3750
@@
 F 0 "C12" V 1721 2700 50  0000 C CNN
 F 1 "100n" V 1812 2700 50  0000 C CNN
-F 2 "" H 1950 2700 50  0001 C CNN
+F 2 "Capacitor_SMD:C_0603_1608Metric" H 1950 2700 50  0001 C CNN
 F 3 "~" H 1950 2700 50  0001 C CNN
 	1    1950 2700
@@
 F 0 "C13" V 1721 4850 50  0000 C CNN
 F 1 "100n" V 1812 4850 50  0000 C CNN
-F 2 "" H 1950 4850 50  0001 C CNN
+F 2 "Capacitor_SMD:C_0603_1608Metric" H 1950 4850 50  0001 C CNN
 F 3 "~" H 1950 4850 50  0001 C CNN
 	1    1950 4850
