File: schematic/devel/detector.sch (KiCad schematic (older format))
At the start: 12 parts, among them U4 OPA4197

Commit message: created S5990 footprint, created pcb layout
Parts:
- D5: footprint (none) -> Sensor_OpticalPosition:S5990
- U4: footprint Package_SO:MSOP-8_3x3mm_P0.65mm -> Package_SO:TSSOP-14_4.4x5mm_P0.65mm
Changed lines of the file:
@@
 F 0 "D5" H 2450 3500 50  0000 L CNN
 F 1 "S599x" H 2400 3400 50  0000 L CNN
-F 2 "" V 2650 3100 50  0001 C CNN
+F 2 "Sensor_OpticalPosition:S5990" V 2650 3100 50  0001 C CNN
 F 3 "" V 2650 3100 50  0001 C CNN
 	1    2550 3200
@@
 F 0 "U4" H 5000 3500 50  0000 C CNN
 F 1 "OPA4197" H 4900 3600 50  0000 C CNN
-F 2 "Package_SO:MSOP-8_3x3mm_P0.65mm" H 4850 3300 50  0001 C CNN
+F 2 "Package_SO:TSSOP-14_4.4x5mm_P0.65mm" H 4850 3300 50  0001 C CNN
 F 3 "~" H 4850 3300 50  0001 C CNN
 	2    4850 3300
@@
 F 0 "U4" H 5000 5100 50  0000 C CNN
 F 1 "OPA4197" H 4900 5200 50  0000 C CNN
-F 2 "Package_SO:MSOP-8_3x3mm_P0.65mm" H 4850 4900 50  0001 C CNN
+F 2 "Package_SO:TSSOP-14_4.4x5mm_P0.65mm" H 4850 4900 50  0001 C CNN
 F 3 "~" H 4850 4900 50  0001 C CNN
 	3    4850 4900
@@
 F 0 "U4" H 3300 3500 50  0000 C CNN
 F 1 "OPA4197" H 3200 3600 50  0000 C CNN
-F 2 "Package_SO:MSOP-8_3x3mm_P0.65mm" H 3150 3300 50  0001 C CNN
+F 2 "Package_SO:TSSOP-14_4.4x5mm_P0.65mm" H 3150 3300 50  0001 C CNN
 F 3 "~" H 3150 3300 50  0001 C CNN
 	1    3150 3300
@@
 F 0 "U4" H 3300 5100 50  0000 C CNN
 F 1 "OPA4197" H 3200 5200 50  0000 C CNN
-F 2 "Package_SO:MSOP-8_3x3mm_P0.65mm" H 3150 4900 50  0001 C CNN
+F 2 "Package_SO:TSSOP-14_4.4x5mm_P0.65mm" H 3150 4900 50  0001 C CNN
 F 3 "~" H 3150 4900 50  0001 C CNN
 	4    3150 4900
@@
 F 0 "U4" V 1325 3750 50  0000 C CNN
 F 1 "OPA4197" V 1416 3750 50  0000 C CNN
-F 2 "Package_SO:MSOP-8_3x3mm_P0.65mm" H 1650 3750 50  0001 C CNN
+F 2 "Package_SO:TSSOP-14_4.4x5mm_P0.65mm" H 1650 3750 50  0001 C CNN
 F 3 "~" H 1650 3750 50  0001 C CNN
 	5    1650 3750
@@
 F 0 "D5" H 4257 3495 50  0000 C CNN
 F 1 "S599x" H 4257 3404 50  0000 C CNN
-F 2 "" H 4200 3200 50  0001 C CNN
+F 2 "Sensor_OpticalPosition:S5990" H 4200 3200 50  0001 C CNN
 F 3 "~" H 4200 3200 50  0001 C CNN
 	2    4250 3200
@@
 F 0 "D5" H 4257 5095 50  0000 C CNN
 F 1 "S599x" H 4257 5004 50  0000 C CNN
-F 2 "" H 4200 4800 50  0001 C CNN
+F 2 "Sensor_OpticalPosition:S5990" H 4200 4800 50  0001 C CNN
 F 3 "~" H 4200 4800 50  0001 C CNN
 	3    4250 4800
@@
 F 0 "D5" H 2557 5095 50  0000 C CNN
 F 1 "S599x" H 2557 5004 50  0000 C CNN
-F 2 "" H 2500 4800 50  0001 C CNN
+F 2 "Sensor_OpticalPosition:S5990" H 2500 4800 50  0001 C CNN
 F 3 "~" H 2500 4800 50  0001 C CNN
 	4    2550 4800
@@
 F 0 "D5" H 8558 3936 50  0000 L CNN
 F 1 "S599x" H 8558 3845 50  0000 L CNN
-F 2 "" H 8450 3850 50  0001 C CNN
+F 2 "Sensor_OpticalPosition:S5990" H 8450 3850 50  0001 C CNN
 F 3 "~" H 8450 3850 50  0001 C CNN
 	5    8500 3850
