File: kicad/experimental/buffer.sch (KiCad schematic (older format))
At the start: 0 parts

Commit message: removed current adc components from experimental kicad design
Parts:
- added C? (x4): 100n, symbol Device:C
- added J?: Power, symbol Connector:Screw_Terminal_01x03
- added J?: Signal Input, symbol Connector:Screw_Terminal_01x04
- added J?: Signal Ouput, symbol Connector:Screw_Terminal_01x04
- added R? (x8): 3k, symbol Device:R
- added R? (x4): 1k, symbol Device:R
- added U? (x6): OPA2197, symbol Device:Opamp_Dual_Generic
Connections:
- new net: R?.1, R?.2, U?.2 (-) (x2)
- new net: R?.1, U?.3 (+) (x2)
- new net: R?.1, U?.5 (+) (x2)
- new net: R?.1, R?.2, U?.6 (-) (x2)
- new net +15V: C?.1, C?.1, J?.1 (Pin_1), U?.8 (V+), U?.8 (V+)
- new net -15V: C?.1, C?.1, J?.3 (Pin_3), U?.4 (V-), U?.4 (V-)
- new net GND: C?.2, C?.2, C?.2, C?.2, J?.2 (Pin_2), R?.2, R?.2, R?.2, R?.2
- new net IX1: J?.4 (Pin_4), R?.2
- new net IX2: J?.3 (Pin_3), R?.2
- new net IY1: J?.2 (Pin_2), R?.2
- new net IY2: J?.1 (Pin_1), R?.2
- new net OX1: J?.4 (Pin_4), R?.1, U?.1
- new net OX2: J?.3 (Pin_3), R?.1, U?.7
- new net OY1: J?.2 (Pin_2), R?.1, U?.1
- new net OY2: J?.1 (Pin_1), R?.1, U?.7
Other:
- note added: "CONVERTER"
- note added: "OX = - IX / 3"
- note added: "POWER"
- note added: "SIGNAL INPUT"
- note added: "SIGNAL OUTPUT"
