File: kicad/2.0.0/arithmetic.sch (KiCad schematic (older format))
At the start: 68 parts, among them J1 Conn_01x03_Male, J2 Conn_01x05_Male, J3 Conn_01x05_Male, J4 Conn_Coaxial, J5 Conn_Coaxial, J6 Conn_Coaxial, U1 LM317, U2 LM337, U3 OPA197xDBV, U4 OPA197xDBV, U5 OPA197xDBV

Commit message: improved arithmetic 2.0.0 pcb
Parts:
- R1, R2, R3, R4: footprint Resistor_SMD:R_0603_1608Metric -> Resistor_SMD:R_1210_3225Metric
- TP4: value DIFFX+ -> DIFFX-
- TP5: value DIFFX- -> DIFFX+
- TP6: value DIFFY- -> DIFFY+
- TP7: value DIFFY+ -> DIFFY-
- TP8: value SUM+ -> SUM-
- TP9: value SUM- -> SUM+
Changed lines of the file:
@@
 F 0 "R4" H 3359 3296 50  0000 L CNN
 F 1 "240" H 3359 3205 50  0000 L CNN
-F 2 "Resistor_SMD:R_0603_1608Metric" H 3300 3250 50  0001 C CNN
+F 2 "Resistor_SMD:R_1210_3225Metric" H 3300 3250 50  0001 C CNN
 F 3 "~" H 3300 3250 50  0001 C CNN
 	1    3300 3250
@@
 F 0 "R3" H 3359 2796 50  0000 L CNN
 F 1 "2.2k" H 3359 2705 50  0000 L CNN
-F 2 "Resistor_SMD:R_0603_1608Metric" H 3300 2750 50  0001 C CNN
+F 2 "Resistor_SMD:R_1210_3225Metric" H 3300 2750 50  0001 C CNN
 F 3 "~" H 3300 2750 50  0001 C CNN
 	1    3300 2750
@@
 F 0 "R2" H 3359 2296 50  0000 L CNN
 F 1 "2.2k" H 3359 2205 50  0000 L CNN
-F 2 "Resistor_SMD:R_0603_1608Metric" H 3300 2250 50  0001 C CNN
+F 2 "Resistor_SMD:R_1210_3225Metric" H 3300 2250 50  0001 C CNN
 F 3 "~" H 3300 2250 50  0001 C CNN
 	1    3300 2250
@@
 F 0 "R1" H 3359 1796 50  0000 L CNN
 F 1 "240" H 3359 1705 50  0000 L CNN
-F 2 "Resistor_SMD:R_0603_1608Metric" H 3300 1750 50  0001 C CNN
+F 2 "Resistor_SMD:R_1210_3225Metric" H 3300 1750 50  0001 C CNN
 F 3 "~" H 3300 1750 50  0001 C CNN
 	1    3300 1750
@@
 P 9000 1150
 F 0 "TP8" V 8954 1338 50  0000 L CNN
-F 1 "SUM+" V 9045 1338 50  0000 L CNN
+F 1 "SUM-" V 9045 1338 50  0000 L CNN
 F 2 "TestPoint:TestPoint_Pad_D1.0mm" H 9200 1150 50  0001 C CNN
 F 3 "~" H 9200 1150 50  0001 C CNN
@@
 P 9050 2300
 F 0 "TP9" H 9108 2418 50  0000 L CNN
-F 1 "SUM-" H 9108 2327 50  0000 L CNN
+F 1 "SUM+" H 9108 2327 50  0000 L CNN
 F 2 "TestPoint:TestPoint_Pad_D1.0mm" H 9250 2300 50  0001 C CNN
 F 3 "~" H 9250 2300 50  0001 C CNN
@@
 P 6300 1150
 F 0 "TP4" V 6254 1338 50  0000 L CNN
-F 1 "DIFFX+" V 6345 1338 50  0000 L CNN
+F 1 "DIFFX-" V 6345 1338 50  0000 L CNN
 F 2 "TestPoint:TestPoint_Pad_D1.0mm" H 6500 1150 50  0001 C CNN
 F 3 "~" H 6500 1150 50  0001 C CNN
@@
 P 6000 3000
 F 0 "TP5" V 5954 3188 50  0000 L CNN
-F 1 "DIFFX-" V 6045 3188 50  0000 L CNN
+F 1 "DIFFX+" V 6045 3188 50  0000 L CNN
 F 2 "TestPoint:TestPoint_Pad_D1.0mm" H 6200 3000 50  0001 C CNN
 F 3 "~" H 6200 3000 50  0001 C CNN
@@
 P 6300 3900
 F 0 "TP7" V 6254 4088 50  0000 L CNN
-F 1 "DIFFY+" V 6345 4088 50  0000 L CNN
+F 1 "DIFFY-" V 6345 4088 50  0000 L CNN
 F 2 "TestPoint:TestPoint_Pad_D1.0mm" H 6500 3900 50  0001 C CNN
 F 3 "~" H 6500 3900 50  0001 C CNN
@@
 P 6000 5750
 F 0 "TP6" V 5954 5938 50  0000 L CNN
-F 1 "DIFFY-" V 6045 5938 50  0000 L CNN
+F 1 "DIFFY+" V 6045 5938 50  0000 L CNN
 F 2 "TestPoint:TestPoint_Pad_D1.0mm" H 6200 5750 50  0001 C CNN
 F 3 "~" H 6200 5750 50  0001 C CNN
